File: Hardware/RTK_mosaic-X5.brd (EAGLE design)
At the start: 151.8 x 101.6 mm, 371 parts, among them J2 MAGJACK-POE, J3 MICRO-SD-PUSH-PUSH-EXT-PIN, J4 Vertical Qwiic Connector, J9 MAGJACK-POE, U1 ESP32-WROVER-IE, U10 POE_PSU-DP990X, U11 SN74AVC4T774PW, U17 URB2405YMD, U2 CH340C, U3 AP7361C-33FGEUDFN-8, U4 TXS0108, U5 TXS0108, U6 AP7361C-33FGEUDFN-8, U7 KSZ8041NLI, U8 MOSAIC-X5X5, U9 KSZ8041NLI

Commit message: V10 PCB - routed
Parts:
- removed D13: LED-RIGHT-ANGLE-PTH-GREEN, SparkFun-LED:CBI-RIGHT-ANGLE-PTH
- removed D15, D16: LED-RIGHT-ANGLE-PTH-BLUE, SparkFun-LED:CBI-RIGHT-ANGLE-PTH
- removed U$105, U$106: (no value), output:BLUE0
- removed U$108: (no value), output:GREEN2
- removed U$109: (no value), output:#_BT_#1
- removed U$110: (no value), output:#_LOG_#5
- removed U$111: (no value), output:#_PVT_#3
- removed U$112: (no value), output:#_RTK_#4
- removed U$115: (no value), output:#_WIFI_#2
- removed U5: TXS0108, SparkFun-IC-Comms:VFQFN-20
- added C37, C63: 0.1uF, SparkFun-Capacitors:0603
- added I2C_IO: JUMPER-SMT_3_2-NC_TRACE_SILK, SparkFun-Jumpers:SMT-JUMPER_3_2-NC_TRACE_SILK
- added PWR: JUMPER-SMT_2_NC_TRACE_SILK, SparkFun-Jumpers:SMT-JUMPER_2_NC_TRACE_SILK
- added R54: 200k, SparkFun-Resistors:0603
- added R55, R56, R57, R58: 4.7k, SparkFun-Resistors:0603
- added R59: 470, SparkFun-Resistors:0603
- added R_SCL_IO, R_SDA_IO: 2.2k, SparkFun-Resistors:0603
- added T1: TRANSFORMER0508, SparkFun-Coils:RFCMF1220100M4T
- added U12: URB2405YMD, SparkFun-IC-Power:URB_YMD-15WR3
- added U13, U14, U15, U16, U18: (no value), 74LVC2T45DC:VSSOP8_(SOT765-1)
- D11: value LED-RIGHT-ANGLE-PTH-AMBER -> Yellow Green Red; device SparkFun-LED:CBI-RIGHT-ANGLE-PTH -> CBI_LED_TRIPLE-3MM:CBI_LED_T-3MM_PTH
- D12: value LED-RIGHT-ANGLE-PTH-BLUE -> Yellow Green Red; device SparkFun-LED:CBI-RIGHT-ANGLE-PTH -> CBI_LED_TRIPLE-3MM:CBI_LED_T-3MM_PTH
- R28, R36, R37, R38, R39: value 1k -> 470
- U$103: device output:BLUE0 -> output:#PWR#0
- U$104: device output:YELLOW1 -> output:#WIFI#1
- U$14: device output:#WIFI#1 -> output:#BT#2
- U$8: device output:#BT#0 -> output:#I�C#0
- U11: value SN74AVC4T774PW -> (none); device SparkFun-IC-Comms:SOP65P640X120-16N -> 74LVC2T45DC:VSSOP8_(SOT765-1)
- U17: value URB2405YMD -> (none); device SparkFun-IC-Power:URB_YMD-15WR3 -> 74LVC2T45DC:VSSOP8_(SOT765-1)
- U4: value TXS0108 -> (none); device SparkFun-IC-Comms:VFQFN-20 -> SparkFun-IC-Comms:VSSOP_8PIN
- moved U$8 121.9 mm to (108.7, 82.6)
- moved U17 91.2 mm to (101.6, 88.9), turned to 90 degrees
- moved U4 58.4 mm to (111.8, 88.9), turned to 90 degrees
- moved R23 52.7 mm to (99.2, 86.0), turned to 180 degrees
- moved U11 40.6 mm to (94.0, 88.9)
- moved LOGO4 23.3 mm to (97.8, 25.4)
- moved U$11 21.5 mm to (23.6, 4.45)
- moved LOG 21.4 mm to (22.9, 4.45)
- moved U$116 19.8 mm to (33.0, 8.89)
- moved R37 19.7 mm to (24.1, 14.0), turned to 270 degrees
- moved LOG_BTN 19.7 mm to (33.0, 2.92)
- moved R27 19.7 mm to (33.0, 14.0), turned to 90 degrees
- moved C18 19.1 mm to (45.1, 16.5)
- moved C20 19.1 mm to (46.7, 16.5)
- moved J3 19.1 mm to (47.0, 2.03)
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Connections:
- removed net ESP32_TX_IO: J13.7, U5.18
- removed net ESP33_RTS_IO: J13.6, U5.17
- removed net ESP34_RX_IO: J13.8, U5.20
- removed net ESP35_CTS_IO: J13.5, U5.16
- removed net MOSAIC_CTS_IO: J5.3, U4.16
- removed net MOSAIC_EVENTA: U11.14, U4.6
- removed net MOSAIC_EVENTA_IO: J5.2, R43.2, U4.15
- removed net MOSAIC_EVENTB: U11.13, U4.7
- removed net MOSAIC_EVENTB_IO: J5.1, R44.2, U4.14
- removed net MOSAIC_LOG_BTN_IO: J13.9, R23.2, R27.2, U4.12
- removed net MOSAIC_PPSO_IO: J13.10, U4.13
- removed net MOSAIC_RTS_IO: J5.4, U4.17
- removed net MOSAIC_RX_IO: J5.6, U4.20
- removed net MOSAIC_TX_IO: J5.5, U4.18
- new net D+_MOSAIC_T: T1.A1, U8.A5
- new net D-_MOSAIC_T: T1.B1, U8.A6
- new net ESP32_TX_O: J13.7, U17.7
- new net ESP33_RTS_O: J13.6, U17.6
- new net ESP34_RX_I: J13.8, U18.7
- new net ESP35_CTS_I: J13.5, U18.6
- new net MOSAIC_CTS_I: J5.3, U15.6
- new net MOSAIC_EVENTA_I: J5.2, R43.2, U13.7
- new net MOSAIC_EVENTB_I: J5.1, R44.2, U13.6
- new net MOSAIC_LOG_BTN_I: J13.9, R23.2, R27.2, U16.7
- new net MOSAIC_RTS_O: J5.4, U14.6
- new net MOSAIC_RX_I: J5.6, U15.7
- new net MOSAIC_TX_O: J5.5, U14.7
- new net N$42: I2C_IO.3, R_SCL_IO.2
- new net N$43: I2C_IO.1, R_SDA_IO.2
- new net N$44: PWR.2, R59.2
- new net N$45: D11.ANODE_3, PWR.1
- new net N$6: C37.1, R54.1, U4.P7, U4.P8
- net 1.8V: now also U11.1, U11.5, U13.1; no longer U11.16, U11.6, U11.7, U11.8
- net 3.3V: now also R57.1, R58.1, R59.1, U17.1, U17.5, U18.1, U4.P2; no longer U5.10, U5.2
- net 3.3V_SW: now also C63.1, R55.1, R56.1, U14.1, U14.5, U15.1, U16.1; no longer R22.1, U11.15, U4.10, U4.2
- net 5V_RAW1: now also U12.4; no longer U17.4
- net D+_MOSAIC: now also T1.A2; no longer U8.A5
- net D-_MOSAIC: now also T1.B2; no longer U8.A6
- net ESP14_SCL: now also U4.P3; no longer U5.6
- net ESP14_SCL_IO: now also R_SCL_IO.1, U4.P6; no longer U5.15
- net ESP15_SDA: now also U4.P4; no longer U5.7
- net ESP15_SDA_IO: now also R_SDA_IO.1, U4.P5; no longer U5.14
- net ESP32_TX: now also U17.2; no longer U5.3
- net ESP33_RTS: now also U17.3; no longer U5.4
- net ESP34_RX: now also U18.2; no longer U5.1
- net ESP35_CTS: now also U18.3; no longer U5.5
- net GND: now also C37.2, C63.2, D11.CATHODE_1, D11.CATHODE_2, D11.CATHODE_3, D12.CATHODE_1, D12.CATHODE_2, D12.CATHODE_3, R22.1, U11.3, U11.4, U12.6, U13.4, U13.5, U14.4, U15.4, U15.5, U16.4, U16.5, U16.6, U17.4, U18.4, U18.5, U4.P1; no longer D11.C, D12.C, D13.C, D15.C, D16.C, U11.1, U11.10, U11.2, U11.9, U17.6, U4.11, U4.EPAD, U5.11, U5.EPAD
- net LINK_ESP32: now also R58.2
- net LINK_MOSAIC: now also R56.2
- net MOSAIC_CTS: now also U15.3; no longer U4.5
- net MOSAIC_EVENTA_1V8: now also U13.2; no longer U11.3
- net MOSAIC_EVENTB_1V8: now also U13.3; no longer U11.4
- net MOSAIC_LOG_BTN: now also U16.2; no longer U4.9
- net MOSAIC_PPSO: now also J13.10, U11.7; no longer U11.12, U4.8
- net MOSAIC_PPSO_1V8: now also U11.2; no longer U11.5
- net MOSAIC_RTS: now also U14.3; no longer U4.4
- net MOSAIC_RX: now also U15.2; no longer U4.1
- net MOSAIC_TX: now also U14.2; no longer U4.3
- net N$17: now also D12.ANODE_3; no longer D13.A
- net N$18: now also D11.ANODE_2; no longer D11.A
- net N$22: now also D11.ANODE_1; no longer D12.A
- net N$35: now also D12.ANODE_2; no longer D15.A
- net N$36: now also D12.ANODE_1; no longer D16.A
- net SPEED_ESP32: now also R57.2
- net SPEED_MOSAIC: now also R55.2
- net VCCIO: now also I2C_IO.2, R54.2, U11.8, U13.8, U14.8, U15.8, U16.8, U17.8, U18.8; no longer U4.19, U5.19
- net VIN1-: now also U12.2; no longer U17.2
- net VIN2+: now also U12.3; no longer U17.3
Routing:
- net MOSAIC_LOG_BTN_IO: track 152.1 -> 0.00 mm, vias 5 -> 0
- net MOSAIC_LOG_BTN_I: track 0.00 -> 137.7 mm, vias 0 -> 4
- net 3.3V: track 309.2 -> 392.5 mm, vias 17 -> 21
- net MOSAIC_PPSO_IO: track 70.2 -> 0.00 mm, vias 1 -> 0
- net D-_MOSAIC: track 64.5 -> 14.4 mm
- net D+_MOSAIC: track 63.5 -> 13.7 mm
- net D-_MOSAIC_T: track 0.00 -> 46.0 mm
- net D+_MOSAIC_T: track 0.00 -> 45.5 mm
- net 3.3V_SW: track 269.0 -> 308.3 mm, vias 11 -> 13
- net MOSAIC_LOG_BTN: track 69.7 -> 37.1 mm
- net VCCIO: track 141.0 -> 171.8 mm, vias 6 -> 12
- net MOSAIC_PPSO_1V8: track 42.3 -> 12.5 mm
- net MOSAIC_EVENTB_IO: track 23.0 -> 0.00 mm, vias 2 -> 0
- net MOSAIC_EVENTA_IO: track 19.0 -> 0.00 mm, vias 2 -> 0
- net MOSAIC_EVENTB_I: track 0.00 -> 16.8 mm, vias 0 -> 2
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Other:
- outline, holes or cut-outs redrawn
- board text added: "v10"
- board text removed: "v01"
