File: Hardware/RTK_mosaic-X5.sch (EAGLE design)
At the start: 244 parts, among them J2 MAGJACK-POE, J3 MICRO-SD-PUSH-PUSH-EXT-PIN, J4 Vertical Qwiic Connector, J9 MAGJACK-POE, U1 ESP32-WROVER-IE, U10 POE_PSU-DP990X, U11 SN74AVC4T774PW, U17 URB2405YMD, U2 CH340C, U3 AP7361C-33FGEUDFN-8, U4 TXS0108, U5 TXS0108, U6 AP7361C-33FGEUDFN-8, U7 KSZ8041NLI, U8 MOSAIC-X5X5, U9 KSZ8041NLI

Commit message: V10 PCB - routed
Parts:
- removed D13: LED-RIGHT-ANGLE-PTH-GREEN, SparkFun-LED:LED-RIGHT-ANGLE-PTH-GREEN
- removed D15, D16: LED-RIGHT-ANGLE-PTH-BLUE, SparkFun-LED:LED-RIGHT-ANGLE-PTH-BLUE
- removed U5: TXS0108, SparkFun-IC-Comms:TXS0108-VFQFN_20
- added C37, C63: 0.1uF, SparkFun-Capacitors:0.1UF-0603-25V-5%
- added I2C_IO: JUMPER-SMT_3_2-NC_TRACE_SILK, SparkFun-Jumpers:JUMPER-SMT_3_2-NC_TRACE_SILK
- added PWR: JUMPER-SMT_2_NC_TRACE_SILK, SparkFun-Jumpers:JUMPER-SMT_2_NC_TRACE_SILK
- added R54: 200k, SparkFun-Resistors:200KOHM-0603-1/10W-1%
- added R55, R56, R57, R58: 4.7k, SparkFun-Resistors:4.7KOHM-0603-1/10W-1%
- added R59: 470, SparkFun-Resistors:470OHM-0603-1/10W-1%
- added R_SCL_IO, R_SDA_IO: 2.2k, SparkFun-Resistors:2.2KOHM-0603-1/10W-1%
- added T1: TRANSFORMER0508, SparkFun-Coils:TRANSFORMER0508
- added U12: URB2405YMD, SparkFun-IC-Power:URB_YMD-15WR3__URB2405YMD-15WR3
- added U13, U14, U15, U16, U18: (no value), 74LVC2T45DC:74LVC2T45DC
- D11: value LED-RIGHT-ANGLE-PTH-AMBER -> Yellow Green Red; device SparkFun-LED:LED-RIGHT-ANGLE-PTH-AMBER -> CBI_LED_TRIPLE-3MM:LED_TRIPLE-3MM_RIGHT-ANGLE_PTH_YELLOW_GREEN_RED
- D12: value LED-RIGHT-ANGLE-PTH-BLUE -> Yellow Green Red; device SparkFun-LED:LED-RIGHT-ANGLE-PTH-BLUE -> CBI_LED_TRIPLE-3MM:LED_TRIPLE-3MM_RIGHT-ANGLE_PTH_YELLOW_GREEN_RED
- R28, R36, R37, R38, R39: value 1k -> 470; device SparkFun-Resistors:1KOHM-0603-1/10W-1% -> SparkFun-Resistors:470OHM-0603-1/10W-1%
- U11: value SN74AVC4T774PW -> (none); device SparkFun-IC-Comms:SN74AVC4T774PW -> 74LVC2T45DC:74LVC2T45DC
- U17: value URB2405YMD -> (none); device SparkFun-IC-Power:URB_YMD-15WR3__URB2405YMD-15WR3 -> 74LVC2T45DC:74LVC2T45DC
- U4: value TXS0108 -> (none); device SparkFun-IC-Comms:TXS0108-VFQFN_20 -> SparkFun-IC-Comms:PCA9306VSSOP_8PIN
Connections:
- removed net ESP32_TX_IO: J13.7, U5.B2
- removed net ESP33_RTS_IO: J13.6, U5.B3
- removed net ESP34_RX_IO: J13.8, U5.B1
- removed net ESP35_CTS_IO: J13.5, U5.B4
- removed net MOSAIC_CTS_IO: J5.3, U4.B4
- removed net MOSAIC_EVENTA: U11.B1, U4.A5
- removed net MOSAIC_EVENTA_IO: J5.2, R43.2, U4.B5
- removed net MOSAIC_EVENTB: U11.B2, U4.A6
- removed net MOSAIC_EVENTB_IO: J5.1, R44.2, U4.B6
- removed net MOSAIC_LOG_BTN_IO: J13.9, R23.2, R27.2, U4.B8
- removed net MOSAIC_PPSO_IO: J13.10, U4.B7
- removed net MOSAIC_RTS_IO: J5.4, U4.B3
- removed net MOSAIC_RX_IO: J5.6, U4.B1
- removed net MOSAIC_TX_IO: J5.5, U4.B2
- new net D+_MOSAIC_T: T1.A1, U8.USB_D+
- new net D-_MOSAIC_T: T1.B1, U8.USB_D-
- new net ESP32_TX_O: J13.7, U17.1B
- new net ESP33_RTS_O: J13.6, U17.2B
- new net ESP34_RX_I: J13.8, U18.1B
- new net ESP35_CTS_I: J13.5, U18.2B
- new net MOSAIC_CTS_I: J5.3, U15.2B
- new net MOSAIC_EVENTA_I: J5.2, R43.2, U13.1B
- new net MOSAIC_EVENTB_I: J5.1, R44.2, U13.2B
- new net MOSAIC_LOG_BTN_I: J13.9, R23.2, R27.2, U16.1B
- new net MOSAIC_RTS_O: J5.4, U14.2B
- new net MOSAIC_RX_I: J5.6, U15.1B
- new net MOSAIC_TX_O: J5.5, U14.1B
- new net N$42: I2C_IO.3, R_SCL_IO.2
- new net N$43: I2C_IO.1, R_SDA_IO.2
- new net N$44: PWR.2, R59.2
- new net N$45: D11.RED_ANODE, PWR.1
- new net N$6: C37.1, R54.1, U4.EN, U4.VREF2
- net 1.8V: now also U11.DIR, U13.VCCA; no longer U11.A4, U11.DIR3, U11.DIR4
- net 3.3V: now also R57.1, R58.1, R59.1, U17.DIR, U17.VCCA, U18.VCCA, U4.VREF1; no longer U5.OE, U5.VCCA
- net 3.3V_SW: now also C63.1, R55.1, R56.1, U14.DIR, U14.VCCA, U15.VCCA, U16.VCCA; no longer R22.1, U11.VCCB, U4.OE, U4.VCCA
- net 5V_RAW1: now also U12.VOUT; no longer U17.VOUT
- net D+_MOSAIC: now also T1.A2; no longer U8.USB_D+
- net D-_MOSAIC: now also T1.B2; no longer U8.USB_D-
- net ESP14_SCL: now also U4.SCL1; no longer U5.A5
- net ESP14_SCL_IO: now also R_SCL_IO.1, U4.SCL2; no longer U5.B5
- net ESP15_SDA: now also U4.SDA1; no longer U5.A6
- net ESP15_SDA_IO: now also R_SDA_IO.1, U4.SDA2; no longer U5.B6
- net ESP32_TX: now also U17.1A; no longer U5.A2
- net ESP33_RTS: now also U17.2A; no longer U5.A3
- net ESP34_RX: now also U18.1A; no longer U5.A1
- net ESP35_CTS: now also U18.2A; no longer U5.A4
- net GND: now also C37.2, C63.2, D11.GREEN_CATHODE, D11.RED_CATHODE, D11.YELLOW_CATHODE, D12.GREEN_CATHODE, D12.RED_CATHODE, D12.YELLOW_CATHODE, R22.1, U11.2A, U12.GND, U13.DIR, U13.GND, U14.GND, U15.DIR, U15.GND, U16.2B, U16.DIR, U16.GND, U18.DIR, U18.GND; no longer D11.C, D12.C, D13.C, D15.C, D16.C, U11.!OE, U11.DIR1, U11.DIR2, U4.EPAD, U5.EPAD, U5.GND
- net LINK_ESP32: now also R58.2
- net LINK_MOSAIC: now also R56.2
- net MOSAIC_CTS: now also U15.2A; no longer U4.A4
- net MOSAIC_EVENTA_1V8: now also U13.1A; no longer U11.A1
- net MOSAIC_EVENTB_1V8: now also U13.2A; no longer U11.A2
- net MOSAIC_LOG_BTN: now also U16.1A; no longer U4.A8
- net MOSAIC_PPSO: now also J13.10, U11.1B; no longer U11.B3, U4.A7
- net MOSAIC_PPSO_1V8: now also U11.1A; no longer U11.A3
- net MOSAIC_RTS: now also U14.2A; no longer U4.A3
- net MOSAIC_RX: now also U15.1A; no longer U4.A1
- net MOSAIC_TX: now also U14.1A; no longer U4.A2
- net N$17: now also D12.RED_ANODE; no longer D13.A
- net N$18: now also D11.GREEN_ANODE; no longer D11.A
- net N$22: now also D11.YELLOW_ANODE; no longer D12.A
- net N$35: now also D12.GREEN_ANODE; no longer D15.A
- net N$36: now also D12.YELLOW_ANODE; no longer D16.A
- net SPEED_ESP32: now also R57.2
- net SPEED_MOSAIC: now also R55.2
- net VCCIO: now also I2C_IO.2, R54.2, U11.VCCB, U13.VCCB, U14.VCCB, U15.VCCB, U16.VCCB, U17.VCCB, U18.VCCB; no longer U4.VCCB, U5.VCCB
- net VIN1-: now also U12.VIN-; no longer U17.VIN-
- net VIN2+: now also U12.VIN+; no longer U17.VIN+
Other:
- note added: "50MHz"
- note added: "ESP32 GPIO0 - Ethernet PHY RMII Reference Clock (50MHz): Take care of the signal integrity of REF_CLK in the hardware design. Keep the trace as short as possible. Keep it away from RF devices and inductor elements."
- note added: "ESP32 IO Level Shifting"
- note added: "Mosaic IO Level Shifting"
- moved on the sheet: ANT1, ANT2, BT, C12, C46, C53, C54, C58, C59, C60, C61, C62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

Commit message: v10 - ready for manufacture
Parts:
- added D13, D15, D16, D18, D19, D20, D21, D22, D23, D24, D25, D26, D27, D28, D29, D30, D31, D32, D33, D34: PESD0402, SparkFun-DiscreteSemi:PESD0402-0402
- added ESP1, ESP2, ESP36, ESP39, RDY1: TEST-POINTPOGO_PTH, SparkFun-Connectors:TEST-POINTPOGO_PTH
Connections:
- new net ESP36: ESP36.1, U1.SENSOR_VP/IA36
- new net ESP39: ESP39.1, U1.SENSOR_VN/IA39
- net 3.3V: now also ESP2.1
- net 3.3V_SW: now also D34.1, RDY1.1
- net ESP14_SCL_IO: now also D26.1
- net ESP15_SDA_IO: now also D25.1
- net ESP32_TX_O: now also D24.1
- net ESP33_RTS_O: now also D23.1
- net ESP34_RX_I: now also D28.1
- net ESP35_CTS_I: now also D27.1
- net GND: now also D13.2, D15.2, D16.2, D18.2, D19.2, D20.2, D21.2, D22.2, D23.2, D24.2, D25.2, D26.2, D27.2, D28.2, D29.2, D30.2, D31.2, D32.2, D33.2, D34.2, ESP1.1
- net MOSAIC_CTS_I: now also D19.1
- net MOSAIC_EVENTA_I: now also D15.1
- net MOSAIC_EVENTB_I: now also D13.1
- net MOSAIC_LOG_BTN_I: now also D18.1
- net MOSAIC_PPSO: now also D16.1
- net MOSAIC_RTS_O: now also D21.1
- net MOSAIC_RX_I: now also D20.1
- net MOSAIC_TX_O: now also D22.1
- net SD_CLK: now also D32.1
- net SD_CMD: now also D33.1
- net SD_DATA: now also D31.1
- net VCCIO: now also D29.1, D30.1
Other:
- note added: "v10"
- note removed: "v01"
- moved on the sheet: C37, C41, C58, C59, C63, I2C_IO, R23, R54, R_SCL_IO, R_SDA_IO, U17, U18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

Commit message: Updates for v1.1 PCB
Other:
- note added: "Ethernet Track Impedance: Differential Pair https://saturnpcb.com/saturn-pcb-toolkit/ Prepreg thickness: 8.3 mil (JLC7628). Er = 4.6 9.0 mil track with 11.0 mil gap (20 mil center to center) = 100 Ohms Each pair should match in length to better than 0.5mm"
- note added: "USB Track Impedance: Differential Pair https://saturnpcb.com/saturn-pcb-toolkit/ Prepreg thickness: 8.3 mil (JLC7628). Er = 4.6 10.5 mil track with 9.5 mil gap (20 mil center to center) = 90 Ohms"
- note added: "v11"
- note removed: "USB Track Impedance: Differential Pair https://saturnpcb.com/saturn-pcb-toolkit/ Prepreg thickness: 0.2mm (7.87 mil). Er = 4.6 10.5 mil track with 9.5 mil gap (20 mil center to center) = 90 Ohms"
- note removed: "v10"
Changed lines of the file:
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@@
 <layer number="255" name="routoute" color="7" fill="1" visible="no" active="no"/>
 </layers>
-<schematic xreflabel="%F%N/%S" xrefpart="/%S.%C%R">
+<schematic xreflabel="%F%N/%S" xrefpart="/%S">
 <attributes>
 </attributes>
@@
 <text x="93.98" y="226.06" size="2.54" layer="94" font="vector" align="top-left">ESP32 USB-C</text>
 <text x="350.52" y="10.16" size="2.54" layer="94" font="vector">Paul Clark</text>
-<text x="421.64" y="7.62" size="2.54" layer="94" font="vector">v10</text>
+<text x="421.64" y="7.62" size="2.54" layer="94" font="vector">v11</text>
 <text x="342.9" y="119.38" size="2.54" layer="94" font="vector" align="top-left">Reset and Boot</text>
 <wire x1="0" y1="175.26" x2="91.44" y2="175.26" width="0.1524" layer="97" style="longdash"/>
@@
 <text x="5.842" y="30.988" size="1.778" layer="97" font="vector" align="top-left">USB Track Impedance: Differential Pair
 https://saturnpcb.com/saturn-pcb-toolkit/
-Prepreg thickness: 0.2mm (7.87 mil). Er = 4.6
+Prepreg thickness: 8.3 mil (JLC7628). Er = 4.6
 10.5 mil track with 9.5 mil gap (20 mil center to center) = 90 Ohms
 </text>
@@
 Keep the trace as short as possible.
 Keep it away from RF devices and inductor elements.</text>
+<text x="112.522" y="18.288" size="1.778" layer="97" font="vector" align="top-left">Ethernet Track Impedance: Differential Pair
+https://saturnpcb.com/saturn-pcb-toolkit/
+Prepreg thickness: 8.3 mil (JLC7628). Er = 4.6
+9.0 mil track with 11.0 mil gap (20 mil center to center) = 100 Ohms
+Each pair should match in length to better than 0.5mm
+</text>
 </plain>
 <instances>
@@
 <text x="182.88" y="256.54" size="1.778" layer="97" font="vector" rot="MR0">50Ω</text>
 <text x="350.52" y="10.16" size="2.54" layer="94" font="vector">Paul Clark</text>
-<text x="421.64" y="7.62" size="2.54" layer="94" font="vector">v10</text>
+<text x="421.64" y="7.62" size="2.54" layer="94" font="vector">v11</text>
 <text x="171.45" y="195.58" size="1.778" layer="97" font="vector">50Ω</text>
 <text x="161.29" y="226.06" size="1.778" layer="97" font="vector">50Ω</text>
