File: Production/RTK_mosaic-X5-Panel.brd (EAGLE design)
At the start: 165.5 x 131.1 mm, 411 parts, among them J2 MAGJACK-POE, J3 MICRO-SD-PUSH-PUSH-EXT-PIN, J4 Vertical Qwiic Connector, J9 MAGJACK-POE, T1 TRANSFORMER0508, U1 ESP32-WROVER-IE, U10 POE_PSU-DP990X, U12 URB2405YMD, U2 CH340C, U3 AP7361C-33FGEUDFN-8, U6 AP7361C-33FGEUDFN-8, U7 KSZ8041NLI, U8 MOSAIC-X5X5, U9 KSZ8041NLI

Commit message: Updates for v1.1 PCB
Parts:
- moved R41 1.65 mm to (137.9, 73.7)
- moved R42 1.65 mm to (139.5, 73.7)
Routing:
- net RD+_MOSAIC: track 28.8 -> 39.4 mm, vias 2 -> 3
- net TD+_MOSAIC: track 25.7 -> 30.2 mm
- net VDDA: track 64.1 -> 68.5 mm
- net RD+_ESP32: track 18.5 -> 22.7 mm
- net VCCA: track 42.7 -> 46.8 mm
- net RD-_ESP32: track 24.0 -> 22.7 mm
- net VIN1+: track 61.4 -> 60.2 mm
- net TD-_MOSAIC: track 29.3 -> 30.2 mm, vias 2 -> 3
- net ESP5_ERST: track 25.9 -> 25.3 mm
- net RD-_MOSAIC: track 40.1 -> 39.4 mm, vias 2 -> 3
- net SPEED_ESP32: track 12.4 -> 13.0 mm
- net TD-_ESP32: track 25.2 -> 25.7 mm, vias 2 -> 3
- net TD+_ESP32: track 25.3 -> 25.7 mm, vias 2 -> 3
- net GND: track 11.4 -> 11.6 mm, vias 426 -> 443
Other:
- board text added: "v11"
- board text removed: "v10"
